File: USB-3.2-gen-1-to-2.5G-Ethernet.kicad_pcb (KiCad board)
At the start: 4 copper layers, 70 x 23 mm, 70 parts, among them U1 RTL8156BG-CG, U2 VL162, U3 HC-RJ45-055-7, U4 TPS62420DRCR, U5 W25Q16BVSSIG, Y1 25Mhz

Commit message: .
Parts:
- removed R8: 1.8M, Resistor_SMD:R_0402_1005Metric
- R5: value 280k -> 270k
- R6: value 910k -> 820k
- moved R6 2.64 mm to (123.1, 98.2), turned to 0 degrees
- moved C5 1.90 mm to (136.6, 101.8), turned to 180 degrees
- moved R7 1.51 mm to (125.1, 97.8), turned to 0 degrees
- moved R4 0.07 mm to (123.7, 103.9)
Connections:
- C6 pad 2: Net-(U4-SW2) -> +0.95V
- R4 pad 1: Net-(U4-SW2) -> +0.95V
- R6 pad 1: Net-(U4-SW1) -> +3.3V
Routing:
- net +0.95V: track 27.5 -> 39.4 mm
- net +3.3V: track 103.5 -> 104.6 mm
- net Net-(U4-ADJ2): track 3.88 -> 2.91 mm
- net Net-(U4-DEF_1): track 3.12 -> 2.60 mm
- net GND: vias 15 -> 14
